File: elec/layout/default/sk6805side.kicad_pcb (KiCad board)
At the start: 2 copper layers, 225.7 x 100.8 mm, 0 parts

Commit message: layout
Parts:
- added C1: Multilayer Ceramic Capacitors MLCC - SMD/SMT 1uF 6.3V 0402 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, lib:C0402, F.Cu at (162.7, 100.3)
- added U1: , lib:LED-SMD_4P-L4.0-W1.4_SK6805SIDE-S, F.Cu at (163.4, 101.6)
Routing:
- net vcc: track 0.00 -> 1.38 mm
- net gnd: track 0.00 -> 1.37 mm
Changed lines of the file:
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@@
   )
   (net 0 "")
+  (net 1 "vcc")
+  (net 2 "gnd")
+  (net 3 "vcc-2")
+  (net 4 "vcc-1")
+  (footprint "lib:LED-SMD_4P-L4.0-W1.4_SK6805SIDE-S" (layer "F.Cu")
+    (at 163.4 101.6)
+    (attr through_hole)
+    (fp_text reference "U1" (at 0 -4.01) (layer "F.SilkS")
+        (effects (font (size 1 1) (thickness 0.15)))
+    )
+    (fp_text value "" (at 0 4.01) (layer "F.Fab")
+        (effects (font (size 1 1) (thickness 0.15)))
+    )
+    (fp_text user "${REFERENCE}" (at 0 0) (layer "F.Fab")
+        (effects (font (size 1 1) (thickness 0.15)))
+    )
+    (fp_line (start -2.06 0.57) (end -2.06 1.14)
+      (stroke (width 0.12) (type solid)) (layer "F.SilkS"))
+    (fp_line (start -2.06 1.14) (end 1.94 1.14)
+      (stroke (width 0.12) (type solid)) (layer "F.SilkS"))
+    (fp_line (start -1.1 -0.21) (end -0.3 -0.21)
+      (stroke (width 0.12) (type solid)) (layer "F.SilkS"))
+    (fp_line (start 0.48 -0.21) (end 0.5 -0.21)
+      (stroke (width 0.12) (type solid)) (layer "F.SilkS"))
+    (fp_line (start 1.18 -0.21) (end 1.23 -0.21)
+      (stroke (width 0.12) (type solid)) (layer "F.SilkS"))
+    (fp_line (start 1.94 1.14) (end 1.94 0.56)
+      (stroke (width 0.12) (type solid)) (layer "F.SilkS"))
+    (fp_circle (center -2.06 -0.21) (end -2.03 -0.21)
+      (stroke (width 0.06) (type solid)) (fill none) (layer "F.Fab"))
+    (pad "1" smd custom (at -1.5 0) (size 0.5 0.4) (layers "F.Cu" "F.Paste" "F.Mask")
+      (net 1 "vcc") (pintype "stereo") (thermal_bridge_angle 45)
+      (options (clearance outline) (anchor rect))
+      (primitives
+        (gr_poly
+          (pts
+            (xy -0.41 -0.52)
+            (xy -0.41 -0.29)
+            (xy -0.82 -0.29)
+            (xy -0.82 0.26)
+            (xy -0.41 0.26)
+            (xy -0.41 0.48)
+            (xy 0.24 0.48)
+            (xy 0.24 -0.52)
+          )
+          (width 0.1) (fill yes))
+      ))
+    (pad "2" smd custom (at 0 0) (size 0.3 0.5) (layers "F.Cu" "F.Paste" "F.Mask")
+      (net 2 "gnd") (pintype "stereo") (thermal_bridge_angle 45)
+      (options (clearance outline) (anchor rect))
+      (primitives
+        (gr_poly
+          (pts
+            (xy -0.14 -0.49)
+            (xy -0.14 0.51)
+            (xy 0.31 0.51)
+            (xy 0.31 -0.49)
+          )
+          (width 0.1) (fill yes))
+      ))
+    (pad "3" smd custom (at 0.85 0) (size 0.2 0.2) (layers "F.Cu" "F.Paste" "F.Mask")
+      (net 3 "vcc-2") (pintype "stereo") (thermal_bridge_angle 45)
+      (options (clearance outline) (anchor rect))
+      (primitives
+        (gr_poly
+          (pts
+            (xy -0.18 -0.49)
+            (xy -0.18 0.51)
+            (xy 0.17 0.51)
+            (xy 0.17 -0.49)
+          )
+          (width 0.1) (fill yes))
+      ))
+    (pad "4" smd custom (at 1.7 0) (size 0.5 0.5) (layers "F.Cu" "F.Paste" "F.Mask")
+      (net 4 "vcc-1") (pintype "stereo") (thermal_bridge_angle 45)
+      (options (clearance outline) (anchor rect))
+      (primitives
+        (gr_poly
+          (pts
+            (xy 0.08 -0.26)
+            (xy 0.08 -0.49)
+            (xy -0.3 -0.49)
+            (xy -0.3 -0.26)
+            (xy -0.31 -0.26)
+            (xy -0.31 0.29)
+            (xy -0.3 0.29)
+            (xy -0.3 0.51)
+            (xy 0.08 0.51)
+            (xy 0.08 0.29)
+            (xy 0.49 0.29)
+            (xy 0.49 -0.26)
+          )
+          (width 0.1) (fill yes))
+      ))
+  )
+  (footprint "lib:C0402" (layer "F.Cu")
+    (at 162.667184 100.338641)
+    (descr "Capacitor SMD 0402 (1005 Metric), square (rectangular) end terminal, IPC_7351 nominal, (Body size source: IPC-SM-782 page 76, https://www.pcb-3d.com/wordpress/wp-content/uploads/ipc-sm-782a_amendment_1_and_2.pdf), generated with kicad-footprint-generator")
+    (tags "capacitor")
+    (attr smd)
+    (fp_text reference "C1" (at 0 -1.16) (layer "F.SilkS")
+        (effects (font (size 1 1) (thickness 0.15)))
+    )
+    (fp_text value "Multilayer Ceramic Capacitors MLCC - SMD/SMT 1uF 6.3V 0402 RoHS" (at 0 1.16) (layer "F.Fab")
+        (effects (font (size 1 1) (thickness 0.15)))
+    )
+    (fp_text user "${REFERENCE}" (at 0 0) (layer "F.Fab")
+        (effects (font (size 0.25 0.25) (thickness 0.04)))
+    )
+    (fp_line (start -0.107836 -0.36) (end 0.107836 -0.36)
+      (stroke (width 0.12) (type solid)) (layer "F.SilkS"))
+    (fp_line (start -0.107836 0.36) (end 0.107836 0.36)
+      (stroke (width 0.12) (type solid)) (layer "F.SilkS"))
+    (fp_line (start -0.91 -0.46) (end 0.91 -0.46)
+      (stroke (width 0.05) (type solid)) (layer "F.CrtYd"))
+    (fp_line (start -0.91 0.46) (end -0.91 -0.46)
+      (stroke (width 0.05) (type solid)) (layer "F.CrtYd"))
+    (fp_line (start 0.91 -0.46) (end 0.91 0.46)
+      (stroke (width 0.05) (type solid)) (layer "F.CrtYd"))
+    (fp_line (start 0.91 0.46) (end -0.91 0.46)
+      (stroke (width 0.05) (type solid)) (layer "F.CrtYd"))
+    (fp_line (start -0.5 -0.25) (end 0.5 -0.25)
+      (stroke (width 0.1) (type solid)) (layer "F.Fab"))
+    (fp_line (start -0.5 0.25) (end -0.5 -0.25)
+      (stroke (width 0.1) (type solid)) (layer "F.Fab"))
+    (fp_line (start 0.5 -0.25) (end 0.5 0.25)
+      (stroke (width 0.1) (type solid)) (layer "F.Fab"))
+    (fp_line (start 0.5 0.25) (end -0.5 0.25)
+      (stroke (width 0.1) (type solid)) (layer "F.Fab"))
+    (pad "1" smd roundrect (at -0.48 0) (size 0.56 0.62) (layers "F.Cu" "F.Paste" "F.Mask") (roundrect_rratio 0.25)
+      (net 1 "vcc") (pintype "stereo"))
+    (pad "2" smd roundrect (at 0.48 0) (size 0.56 0.62) (layers "F.Cu" "F.Paste" "F.Mask") (roundrect_rratio 0.25)
+      (net 2 "gnd") (pintype "stereo"))
+    (model "${KICAD6_3DMODEL_DIR}/Capacitor_SMD.3dshapes/C_0402_1005Metric.wrl"
+      (offset (xyz 0 0 0))
+      (scale (xyz 1 1 1))
+      (rotate (xyz 0 0 0))
+    )
+  )
   (gr_circle (center 225.62 81.79) (end 227.32 81.79)
     (stroke (width 0.1) (type solid)) (fill none) (layer "Edge.Cuts"))
@@
       (xy 69.100734 49.778315)
     )
-    (stroke (width 0) (type solid)) (fill none) (layer "Edge.Cuts"))
+    (stroke (width 0.1) (type solid)) (fill none) (layer "Edge.Cuts"))
   (gr_arc (start 261.62 113.79) (mid 260.448427 116.618427) (end 257.62 117.79)
     (stroke (width 0.1) (type solid)) (layer "Edge.Cuts"))
@@
     (effects (font (size 2 2) (thickness 0.1)) (justify left bottom))
   )
+  (segment (start 161.9 100.625825) (end 162.187184 100.338641) (width 0.25) (layer "F.Cu") (net 1))
+  (segment (start 161.9 101.6) (end 161.9 100.625825) (width 0.25) (layer "F.Cu") (net 1))
+  (segment (start 163.4 101.6) (end 163.4 100.591457) (width 0.25) (layer "F.Cu") (net 2))
+  (segment (start 163.4 100.591457) (end 163.147184 100.338641) (width 0.25) (layer "F.Cu") (net 2))
   (group "" (id 6c1ef9f7-0f34-47bb-ac1a-76df23fb396e)
     (members
